Commit message: Updated vla_kinova.urdf.xacro
Updated the file to mirror the functioning of the original kinova.urdf.xacro file instead of simply wrapping it, thus exposing more arguments while making it possible to fix the gazebo camera pose from our package

File: urdf/vla_kinova.urdf.xacro (robot description, xacro)
@@ -11,5 +11,141 @@
   <xacro:arg name="simulation_controllers" default="" />
   <xacro:arg name="gripper" default="" />
-  <xacro:include filename="$(find kortex_description)/robots/kinova.urdf.xacro" />
+  <xacro:arg name="username" default="admin" />
+  <xacro:arg name="password" default="admin" />
+  <xacro:arg name="port" default="10000" />
+  <xacro:arg name="port_realtime" default="10001" />
+  <xacro:arg name="session_inactivity_timeout_ms" default="60000" />
+  <xacro:arg name="connection_inactivity_timeout_ms" default="2000" />
+  <xacro:arg name="gripper_joint_name" default="finger_joint" />
+  <xacro:arg name="gripper_max_velocity" default="100.0" />
+  <xacro:arg name="gripper_max_force" default="100.0" />
+  <xacro:arg name="use_internal_bus_gripper_comm" default="false" />
+  <xacro:arg name="use_fake_hardware" default="false" />
+  <xacro:arg name="fake_sensor_commands" default="false" />
+  <xacro:arg name="sim_isaac" default="false" />
+  <xacro:arg name="use_external_cable" default="false" />
+  <xacro:arg name="gazebo_renderer" default="ogre"/>
+  <xacro:arg name="camera_width" default="640"/>
+  <xacro:arg name="camera_height" default="480"/>
+  <xacro:arg name="camera_fps" default="6"/>
+  <xacro:arg name="moveit_active" default="false"/>
+  <xacro:arg name="initial_positions_file" default="$(find kortex_description)/config/initial_positions.yaml"/>
+  <!-- convert to property to use substitution in function -->
+  <xacro:property name="initial_positions_file" default="$(arg initial_positions_file)"/>
+  <!-- Import the core robot macro instead of the stock kinova.urdf.xacro -->
+  <xacro:include filename="$(find kortex_description)/robots/kortex_robot.xacro" />
+  <!-- Create link fixed to the "world" -->
+  <link name="world" />
+  <!-- Load the robot -->
+  <xacro:load_robot
+    parent="world"
+    arm="$(arg arm)"
+    gripper="$(arg gripper)"
+    gripper_joint_name="$(arg gripper_joint_name)"
+    gripper_max_velocity="$(arg gripper_max_velocity)"
+    gripper_max_force="$(arg gripper_max_force)"
+    dof="$(arg dof)"
+    vision="$(arg vision)"
+    robot_ip="$(arg robot_ip)"
+    username="$(arg username)"
+    password="$(arg password)"
+    port="$(arg port)"
+    port_realtime="$(arg port_realtime)"
+    session_inactivity_timeout_ms="$(arg session_inactivity_timeout_ms)"
+    connection_inactivity_timeout_ms="$(arg connection_inactivity_timeout_ms)"
+    use_internal_bus_gripper_comm="$(arg use_internal_bus_gripper_comm)"
+    prefix="$(arg prefix)"
+    use_fake_hardware="$(arg use_fake_hardware)"
+    fake_sensor_commands="$(arg fake_sensor_commands)"
+    sim_gazebo="$(arg sim_gazebo)"
+    sim_ignition="$(arg sim_ignition)"
+    sim_isaac="$(arg sim_isaac)"
+    use_external_cable="$(arg use_external_cable)"
+    initial_positions="${xacro.load_yaml(initial_positions_file)}"
+    moveit_active="$(arg moveit_active)">
+    <origin xyz="0 0 0" rpy="0 0 0" />
+  </xacro:load_robot>
+  <!-- Local definition of Gazebo plugins and sensor overrides -->
+  <xacro:if value="$(arg sim_ignition)">
+    <gazebo>
+      <plugin filename="libign_ros2_control-system.so" name="ign_ros2_control::IgnitionROS2ControlPlugin">
+        <parameters>$(arg simulation_controllers)</parameters>
+        <controller_manager_node_name>$(arg prefix)controller_manager</controller_manager_node_name>
+      </plugin>
+      <plugin filename="libignition-gazebo-sensors-system.so" name="ignition::gazebo::systems::Sensors">
+        <render_engine>$(arg gazebo_renderer)</render_engine>
+      </plugin>
+    </gazebo>
+    <gazebo reference="$(arg prefix)camera_color_frame">
+      <sensor name="camera_sensor" type="rgbd_camera">
+        <!-- GAZEBO CAMERA POSE CORRECTION -->
+        <pose>0 0 0 1.57079632679 -1.57079632679 0</pose>
+        <camera>
+          <horizontal_fov>1.047</horizontal_fov>
+          <image>
+            <width>$(arg camera_width)</width>
+            <height>$(arg camera_height)</height>
+            <format>RGB_INT8</format>
+          </image>
+          <clip>
+            <near>0.1</near>
+            <far>5</far>
+          </clip>
+          <distortion>
+            <k1>0.0</k1>
+            <k2>0.0</k2>
+            <k3>0.0</k3>
+            <p1>0.0</p1>
+            <p2>0.0</p2>
+            <center>0.5 0.5</center>
+          </distortion>
+          <lens>
+            <intrinsics>
+              <fx>554.25469</fx>
+              <fy>554.25469</fy>
+              <cx>320.5</cx>
+              <cy>240.5</cy>
+              <s>0</s>
+            </intrinsics>
+            <projection>
+              <p_fx>554.25469</p_fx>
+              <p_fy>554.25469</p_fy>
+              <p_cx>320.5</p_cx>
+              <p_cy>240.5</p_cy>
+              <tx>0</tx>
+              <ty>0</ty>
+            </projection>
+          </lens>
+          <noise>
+            <type>gaussian</type>
+            <mean>0</mean>
+            <stddev>0.00</stddev>
+          </noise>
+          <depth_camera>
+            <clip>
+              <near>0.25</near>
+              <far>5</far>
+            </clip>
+          </depth_camera>
+          <optical_frame_id>$(arg prefix)color_optical_frame</optical_frame_id>
+        </camera>
+        <ignition_frame_id>$(arg prefix)camera_color_frame</ignition_frame_id>
+        <always_on>1</always_on>
+        <update_rate>$(arg camera_fps)</update_rate>
+        <visualize>true</visualize>
+        <topic>wrist_mounted_camera</topic>
+        <enable_metrics>false</enable_metrics>
+      </sensor>
+    </gazebo>
+  </xacro:if>
+  <!-- Legacy Gazebo Classic support (optional, matching stock wrapper) -->
+  <xacro:if value="$(arg sim_gazebo)">
+    <gazebo>
+      <plugin filename="libgazebo_ros2_control.so" name="gazebo_ros2_control">
+        <parameters>$(arg simulation_controllers)</parameters>
+      </plugin>
+    </gazebo>
+  </xacro:if>
+  <!-- Custom camera frame definitions for when vision module is not used -->
   <xacro:if value="${'$(arg vision)' == 'false'}">
     <link name="$(arg prefix)camera_link">

Commit message: Computed and added approximations for objects inertial properties using blender
- Analyzed meshes in blender and computed approximated inertial parameters
- Found a partial fix for the broken gripper spawning but which breaks the gripper control instead

File: urdf/vla_kinova.urdf.xacro (robot description, xacro)
@@ -66,4 +66,22 @@
     <origin xyz="0 0 0" rpy="0 0 0" />
   </xacro:load_robot>
+  <!-- FORCE GRIPPER TO SPAWN OPEN (0.0) TO PREVENT MIMIC JOINT EXPLOSION -->
+  <!-- This overrides the 0.7929 default in the robotiq_description -->
+  <!-- <ros2_control name="gen3_gripper_fix" type="system">
+    <hardware>
+      <xacro:if value="$(arg sim_ignition)">
+        <plugin>ign_ros2_control/IgnitionSystem</plugin>
+      </xacro:if>
+      <xacro:unless value="$(arg sim_ignition)">
+        <plugin>mock_components/GenericSystem</plugin>
+      </xacro:unless>
+    </hardware>
+    <joint name="$(arg prefix)robotiq_85_left_knuckle_joint">
+      <command_interface name="position" />
+      <state_interface name="position">
+        <param name="initial_value">0.0</param>
+      </state_interface>
+    </joint>
+  </ros2_control> -->
   <!-- Local definition of Gazebo plugins and sensor overrides -->
   <xacro:if value="$(arg sim_ignition)">

Commit message: Added external camera, publishing on topic /external_camera
Notes:
- Couldn't use a real wideangle camera plugin, as it is not available on Ignition Fortress

File: urdf/vla_kinova.urdf.xacro (robot description, xacro)
@@ -35,4 +35,6 @@
   <!-- Import the core robot macro instead of the stock kinova.urdf.xacro -->
   <xacro:include filename="$(find kortex_description)/robots/kortex_robot.xacro" />
+  <!-- Import external camera -->
+  <xacro:include filename="$(find vla_simulation)/urdf/external_camera.urdf.xacro" />
   <!-- Create link fixed to the "world" -->
   <link name="world" />
@@ -66,22 +68,9 @@
     <origin xyz="0 0 0" rpy="0 0 0" />
   </xacro:load_robot>
-  <!-- FORCE GRIPPER TO SPAWN OPEN (0.0) TO PREVENT MIMIC JOINT EXPLOSION -->
-  <!-- This overrides the 0.7929 default in the robotiq_description -->
-  <!-- <ros2_control name="gen3_gripper_fix" type="system">
-    <hardware>
-      <xacro:if value="$(arg sim_ignition)">
-        <plugin>ign_ros2_control/IgnitionSystem</plugin>
-      </xacro:if>
-      <xacro:unless value="$(arg sim_ignition)">
-        <plugin>mock_components/GenericSystem</plugin>
-      </xacro:unless>
-    </hardware>
-    <joint name="$(arg prefix)robotiq_85_left_knuckle_joint">
-      <command_interface name="position" />
-      <state_interface name="position">
-        <param name="initial_value">0.0</param>
-      </state_interface>
-    </joint>
-  </ros2_control> -->
+  <!-- External Camera -->
+  <xacro:external_camera prefix="$(arg prefix)" parent="$(arg prefix)base_link">
+    <origin xyz="0.8 0.0 0.8" rpy="0 0.872665 3.14159265359" />
+    <!-- camera tilted 50 degrees, 0.8 meters in front and 0.8 meters higher than the robot's base -->
+  </xacro:external_camera>
   <!-- Local definition of Gazebo plugins and sensor overrides -->
   <xacro:if value="$(arg sim_ignition)">
